Commit message: added slides and some modification to urdf file

File: myur5_description/urdf/myur5.urdf.xacro (robot description, xacro)
@@ -13,6 +13,6 @@
         <cylinder radius="0.1" length="1"/>
       </geometry>
-      <material name="Gray">
-        <color rgba="0.5 0.5 0.5 0" />
+      <material name="Orange">
+        <color rgba="${255/255} ${108/255} ${10/255} 1.0"/>
       </material>
     </visual>
