Commit message: Including part 2 of the series

File: myur5_description/urdf/myur5_2.urdf.xacro (robot description, xacro)
@@ -1,5 +1,5 @@
 <?xml version="1.0"?>
 <robot xmlns:xacro="http://wiki.ros.org/xacro" name="myur5">
-  <xacro:include filename="$(find myur5_description)/urdf/myur5.gazebo" />
+  <xacro:include filename="$(find myur5_description)/urdf/myur5.gazebo2" />
   <xacro:include filename="$(find myur5_description)/urdf/materials.xacro" />
   <link name="world"/>
@@ -33,5 +33,5 @@
   <xacro:arg name="transmission_hw_interface" default="hardware_interface/PositionJointInterface"/>
   <!-- common stuff -->
-  <xacro:include filename="$(find ur_description)/urdf/common.gazebo.xacro" />
+  <!--xacro:include filename="$(find ur_description)/urdf/common.gazebo.xacro" /-->
   <!-- ur5 -->
   <xacro:include filename="$(find ur_description)/urdf/ur5.urdf.xacro" />
@@ -47,5 +47,5 @@
   <xacro:property name="camera_width" value="0.04" />
   <joint name="camera_joint" type="fixed">
-    <origin xyz="0 0.05 0.07" rpy="0 0 1.57"/>
+    <origin xyz="${camera_width} 0.05 0.01" rpy="0 0 1.57"/>
     <parent link="wrist_3_link"/>
     <child link="camera_link"/>
